File: DPM.kicad_pcb (KiCad board)
At the start: 2 copper layers, 95.9 x 90.2 mm, 15 parts, among them U1 74HC590A, U2 74HC682

Commit message: git-svn-id: file:///D%5C00%20-%20Dev%20&%20Calculs%5CRepoTortoiseSVN_PCB%5CD-DPM/trunk@9 f29d8339-a183-0348-962e-9e4594cf8312
Parts:
- U1: value 74HC590A -> 74HC590
- moved C_1 73.0 mm to (64.1, 122.8)
- moved C_2 73.0 mm to (79.3, 122.8)
- moved LDL1 73.0 mm to (71.7, 126.0)
- moved F1 73.0 mm to (63.8, 128.5)
- moved J_VIN_0 73.0 mm to (58.4, 128.5)
- moved LED1 69.5 mm to (59.5, 116.9)
- moved R5 69.4 mm to (65.2, 116.8), turned to 180 degrees
- moved U1 21.5 mm to (88.3, 91.4), turned to 180 degrees
- moved U2 15.4 mm to (101.6, 73.7)
Connections:
- U1 pad 1: unconnected-(U1-Q1-Pad1) -> Net-(U1-Q1)
- U1 pad 12: unconnected-(U1-~{CE}-Pad12) -> Ground
- U1 pad 15: unconnected-(U1-Q0-Pad15) -> Net-(U1-Q0)
- U1 pad 16: unconnected-(U1-VCC-Pad16) -> VCC
- U1 pad 2: unconnected-(U1-Q2-Pad2) -> Net-(U1-Q2)
- U1 pad 3: unconnected-(U1-Q3-Pad3) -> Net-(U1-Q3)
- U1 pad 4: unconnected-(U1-Q4-Pad4) -> Net-(U1-Q4)
- U1 pad 5: unconnected-(U1-Q5-Pad5) -> Net-(U1-Q5)
- U1 pad 6: unconnected-(U1-Q6-Pad6) -> Net-(U1-Q6)
- U1 pad 7: unconnected-(U1-Q7-Pad7) -> Net-(U1-Q7)
- U2 pad 11: unconnected-(U2-P4-Pad11) -> Net-(U1-Q3)
- U2 pad 13: unconnected-(U2-P5-Pad13) -> Net-(U1-Q2)
- U2 pad 15: unconnected-(U2-P6-Pad15) -> Net-(U1-Q1)
- U2 pad 17: unconnected-(U2-P7-Pad17) -> Net-(U1-Q0)
- U2 pad 2: unconnected-(U2-P0-Pad2) -> Net-(U1-Q7)
- U2 pad 20: unconnected-(U2-VCC-Pad20) -> VCC
- U2 pad 4: unconnected-(U2-P1-Pad4) -> Net-(U1-Q6)
- U2 pad 6: unconnected-(U2-P2-Pad6) -> Net-(U1-Q5)
- U2 pad 8: unconnected-(U2-P3-Pad8) -> Net-(U1-Q4)
Routing:
- net Ground: track 0.00 -> 527.6 mm
- net VCC: track 8.84 -> 154.3 mm
- net Net-(U1-Q1): track 0.00 -> 39.9 mm
- net Net-(U1-Q0): track 0.00 -> 37.6 mm
- net Net-(U1-Q2): track 0.00 -> 33.6 mm
- net Net-(U1-Q3): track 0.00 -> 25.2 mm
- net VBatt: track 11.5 -> 29.7 mm
- net Net-(U1-Q4): track 0.00 -> 16.5 mm
- net Net-(U1-Q5): track 0.00 -> 15.4 mm
- net Net-(U1-Q6): track 0.00 -> 14.4 mm
- net Net-(U1-Q7): track 0.00 -> 13.3 mm
- net /Vin: track 0.00 -> 8.03 mm
- net Net-(LED1-A): track 0.00 -> 2.72 mm

Commit message: git-svn-id: file:///D%5C00%20-%20Dev%20&%20Calculs%5CRepoTortoiseSVN_PCB%5CD-DPM/trunk@12 f29d8339-a183-0348-962e-9e4594cf8312
Parts:
- added J1: Conn_01x08, Connector_PinHeader_2.54mm:PinHeader_1x08_P2.54mm_Vertical, F.Cu at (81.3, 50.8)
- added U4: MCP23017_SP, Package_DIP:DIP-28_W7.62mm_Socket_LongPads, F.Cu at (119.4, 58.4)
- moved U2 17.0 mm to (94.0, 58.4)
- moved U1 14.5 mm to (81.3, 78.7)
Connections:
- PCIe_CAN_1 pad 4: /Connection PCI CAN Express/OSC1 -> Clock
- PCIe_SPI_1 pad 11: /Connection PCI CAN Express/I2C_SDA -> SDA
- PCIe_SPI_1 pad 9: /Connection PCI CAN Express/I2C_SCL -> SCL
- U1 pad 10: unconnected-(U1-~{CCLR}-Pad10) -> VCC
- U1 pad 11: unconnected-(U1-CCLK-Pad11) -> Clock
- U1 pad 13: unconnected-(U1-RCLK-Pad13) -> Clock
- U1 pad 14: unconnected-(U1-~{OE}-Pad14) -> Ground
- U2 pad 1: unconnected-(U2-~{P>Q}-Pad1) -> Net-(J1-Pin_1)
- U2 pad 12: unconnected-(U2-Q4-Pad12) -> Net-(U2-Q4)
- U2 pad 14: unconnected-(U2-Q5-Pad14) -> Net-(U2-Q5)
- U2 pad 16: unconnected-(U2-Q6-Pad16) -> Net-(U2-Q6)
- U2 pad 18: unconnected-(U2-Q7-Pad18) -> Net-(U2-Q7)
- U2 pad 3: unconnected-(U2-Q0-Pad3) -> Net-(U2-Q0)
- U2 pad 5: unconnected-(U2-Q1-Pad5) -> Net-(U2-Q1)
- U2 pad 7: unconnected-(U2-Q2-Pad7) -> Net-(U2-Q2)
- U2 pad 9: unconnected-(U2-Q3-Pad9) -> Net-(U2-Q3)
Routing:
- net Ground: track 527.6 -> 83.9 mm
- net VCC: track 154.3 -> 0.00 mm
- net SCL: track 0.00 -> 80.5 mm
- net SDA: track 0.00 -> 74.7 mm
- net Net-(J1-Pin_6): track 0.00 -> 69.2 mm
- net Net-(J1-Pin_7): track 0.00 -> 64.1 mm
- net Net-(J1-Pin_8): track 0.00 -> 59.0 mm
- net Net-(U2-Q7): track 0.00 -> 44.5 mm
- net Clock: track 0.00 -> 40.4 mm
- net Net-(U2-Q6): track 0.00 -> 38.0 mm
- net Net-(U2-Q5): track 0.00 -> 31.4 mm
- net Net-(U2-Q3): track 0.00 -> 30.7 mm
- net Net-(U2-Q2): track 0.00 -> 29.6 mm
- net Net-(U2-Q1): track 0.00 -> 28.6 mm
- net Net-(U2-Q0): track 0.00 -> 28.2 mm
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- added copper zone on F.Cu, net VCC
- removed copper zone on F.Cu, net Ground

Commit message: DPM et DDPM implémentés Mouais bof pour ajouter ma DPM en code Gray
Sinon OK Tiers pour en faire la branche 1

git-svn-id: file:///D%5C00%20-%20Dev%20&%20Calculs%5CRepoTortoiseSVN_PCB%5CD-DPM/trunk@14 f29d8339-a183-0348-962e-9e4594cf8312
Parts:
- added U3: ADG333A, Package_DIP:DIP-20_W7.62mm_Socket_LongPads, F.Cu at (109.2, 109.2)
- added U5: ADG333A, Package_DIP:DIP-20_W7.62mm_Socket_LongPads, F.Cu at (109.2, 94.0)
- moved U2 25.4 mm to (109.2, 78.7), turned to -90 degrees
- moved J1 17.8 mm to (99.1, 50.8), turned to -90 degrees
- moved U1 13.7 mm to (76.2, 91.4)
- moved U4 12.7 mm to (106.7, 58.4), turned to -90 degrees
Connections:
- net Net-(J1-Pin_1) renamed DPM
- net Net-(J1-Pin_7) renamed I2C_A1
- net Net-(U1-Q0) renamed /Q0
- net Net-(U1-Q1) renamed /Q1
- net Net-(U1-Q2) renamed /Q2
- net Net-(U1-Q3) renamed /Q3
- net Net-(U1-Q4) renamed /Q4
- net Net-(U1-Q5) renamed /Q5
- net Net-(U1-Q6) renamed /Q6
- net Net-(U1-Q7) renamed /Q7
- J1 pad 2: unconnected-(J1-Pin_2-Pad2) -> Dyadic DPM
- J1 pad 3: unconnected-(J1-Pin_3-Pad3) -> Gray DPM
- J1 pad 6: Net-(J1-Pin_6) -> I2C_A2
- J1 pad 8: Net-(J1-Pin_8) -> I2C_A0
- U2 pad 12: Net-(U2-Q4) -> /B4
- U2 pad 14: Net-(U2-Q5) -> /B5
- U2 pad 16: Net-(U2-Q6) -> /B6
- U2 pad 18: Net-(U2-Q7) -> /B7
- U2 pad 3: Net-(U2-Q0) -> /B0
- U2 pad 5: Net-(U2-Q1) -> /B1
- U2 pad 7: Net-(U2-Q2) -> /B2
- U2 pad 9: Net-(U2-Q3) -> /B3
- U4 pad 1: Net-(U2-Q0) -> unconnected-(U4-GPB0-Pad1)
- U4 pad 15: Net-(J1-Pin_6) -> I2C_A0
- U4 pad 17: Net-(J1-Pin_8) -> I2C_A2
- U4 pad 2: Net-(U2-Q1) -> unconnected-(U4-GPB1-Pad2)
- U4 pad 21: unconnected-(U4-GPA0-Pad21) -> /B0
- U4 pad 22: unconnected-(U4-GPA1-Pad22) -> /B1
- U4 pad 23: unconnected-(U4-GPA2-Pad23) -> /B2
- U4 pad 24: unconnected-(U4-GPA3-Pad24) -> /B3
- U4 pad 25: unconnected-(U4-GPA4-Pad25) -> /B4
- U4 pad 26: unconnected-(U4-GPA5-Pad26) -> /B5
- U4 pad 27: unconnected-(U4-GPA6-Pad27) -> /B6
- U4 pad 28: unconnected-(U4-GPA7-Pad28) -> /B7
- U4 pad 3: Net-(U2-Q2) -> unconnected-(U4-GPB2-Pad3)
- U4 pad 4: Net-(U2-Q3) -> unconnected-(U4-GPB3-Pad4)
- U4 pad 5: Net-(U2-Q4) -> unconnected-(U4-GPB4-Pad5)
- U4 pad 6: Net-(U2-Q5) -> unconnected-(U4-GPB5-Pad6)
- U4 pad 7: Net-(U2-Q6) -> unconnected-(U4-GPB6-Pad7)
- U4 pad 8: Net-(U2-Q7) -> unconnected-(U4-GPB7-Pad8)
Routing:
- net Ground: track 83.9 -> 421.7 mm
- net VCC: track 0.00 -> 326.1 mm
- net /B5: track 0.00 -> 90.9 mm
- net /B3: track 0.00 -> 85.5 mm
- net /Q7: track 13.8 -> 97.1 mm
- net /B1: track 0.00 -> 82.1 mm
- net /B0: track 0.00 -> 80.8 mm
- net Dyadic DPM: track 0.00 -> 79.4 mm
- net /B6: track 0.00 -> 72.4 mm
- net Net-(J1-Pin_6): track 69.2 -> 0.00 mm
- net /B2: track 0.00 -> 64.1 mm
- net /Q6: track 12.7 -> 73.4 mm
- net Net-(J1-Pin_8): track 59.0 -> 0.00 mm
- net /Q5: track 13.8 -> 70.2 mm
- net /Q4: track 14.8 -> 71.0 mm
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
Commit message: - Ajout de screenshots de doc
git-svn-id: file:///D%5C00%20-%20Dev%20&%20Calculs%5CRepoTortoiseSVN_PCB%5CD-DPM/trunk@15 f29d8339-a183-0348-962e-9e4594cf8312
Connections:
- U2 pad 12: /B4 -> Net-(U2-Q4)
- U2 pad 14: /B5 -> Net-(U2-Q5)
- U2 pad 16: /B6 -> Net-(U2-Q6)
- U2 pad 18: /B7 -> Net-(U2-Q7)
- U2 pad 3: /B0 -> Net-(U2-Q0)
- U2 pad 5: /B1 -> Net-(U2-Q1)
- U2 pad 7: /B2 -> Net-(U2-Q2)
- U2 pad 9: /B3 -> Net-(U2-Q3)
- U4 pad 1: unconnected-(U4-GPB0-Pad1) -> /B0
- U4 pad 2: unconnected-(U4-GPB1-Pad2) -> /B1
- U4 pad 21: /B0 -> Net-(U2-Q0)
- U4 pad 22: /B1 -> Net-(U2-Q1)
- U4 pad 23: /B2 -> Net-(U2-Q2)
- U4 pad 24: /B3 -> Net-(U2-Q3)
- U4 pad 25: /B4 -> Net-(U2-Q4)
- U4 pad 26: /B5 -> Net-(U2-Q5)
- U4 pad 27: /B6 -> Net-(U2-Q6)
- U4 pad 28: /B7 -> Net-(U2-Q7)
- U4 pad 3: unconnected-(U4-GPB2-Pad3) -> /B2
- U4 pad 4: unconnected-(U4-GPB3-Pad4) -> /B3
- U4 pad 5: unconnected-(U4-GPB4-Pad5) -> /B4
- U4 pad 6: unconnected-(U4-GPB5-Pad6) -> /B5
- U4 pad 7: unconnected-(U4-GPB6-Pad7) -> /B6
- U4 pad 8: unconnected-(U4-GPB7-Pad8) -> /B7
